File: KICAD/ATTN_unit.kicad_sch (KiCad schematic)
At the start: 4 parts, among them U1 DM-OLED096-636, U2 HLK-LD2410C, U4 ESP32-DEVKITC-32E

Commit message: Add files via upload
Parts:
- added SW1: SW_Push, Button_Switch_THT:SW_Tactile_Straight_KSA0Axx1LFTR, symbol Switch:SW_Push
Connections:
- net at KY038.2 (GND), U1.1 (GND), U2.4 (GND)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: now also SW1.2
- net at U4.J3_14 (IO0): now also SW1.1
Changed lines of the file:
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@@
 	(paper "A4")
+	(junction
+		(at 214.63 58.42)
+		(diameter 0)
+		(color 0 0 0 0)
+	)
 	(junction
 		(at 138.43 66.04)
@@
 	(wire
 		(pts
+			(xy 245.11 86.36) (xy 245.11 58.42)
+		)
+		(stroke
+			(width 0)
+			(type default)
+		)
+	)
+	(wire
+		(pts
 			(xy 123.19 110.49) (xy 123.19 58.42)
 		)
@@
 	(wire
 		(pts
+			(xy 234.95 86.36) (xy 234.95 99.06)
+		)
+		(stroke
+			(width 0)
+			(type default)
+		)
+	)
+	(wire
+		(pts
 			(xy 214.63 58.42) (xy 214.63 66.04)
 		)
@@
 	(wire
 		(pts
+			(xy 234.95 99.06) (xy 214.63 99.06)
+		)
+		(stroke
+			(width 0)
+			(type default)
+		)
+	)
+	(wire
+		(pts
 			(xy 125.73 66.04) (xy 138.43 66.04)
 		)
@@
 		(pts
 			(xy 119.38 97.79) (xy 119.38 91.44)
+		)
+		(stroke
+			(width 0)
+			(type default)
+		)
+	)
+	(wire
+		(pts
+			(xy 214.63 58.42) (xy 245.11 58.42)
 		)
 		(stroke
@@
 					(unit 1)
 				)
+			)
+		)
+	)
+	(symbol
+		(lib_id "Switch:SW_Push")
+		(at 240.03 86.36 0)
+		(unit 1)
+		(body_style 1)
+		(exclude_from_sim no)
+		(in_bom yes)
+		(on_board yes)
+		(in_pos_files yes)
+		(dnp no)
+		(fields_autoplaced yes)
+		(property "Reference" "SW1"
+			(at 240.03 78.74 0)
+			(show_name no)
+			(do_not_autoplace no)
+			(effects
+				(font
+					(size 1.27 1.27)
+				)
+			)
+		)
+		(property "Value" "SW_Push"
+			(at 240.03 81.28 0)
+			(show_name no)
+			(do_not_autoplace no)
+			(effects
+				(font
+					(size 1.27 1.27)
+				)
+			)
+		)
+		(property "Footprint" "Button_Switch_THT:SW_Tactile_Straight_KSA0Axx1LFTR"
+			(at 240.03 81.28 0)
+			(hide yes)
+			(show_name no)
+			(do_not_autoplace no)
+			(effects
+				(font
+					(size 1.27 1.27)
+				)
+			)
+		)
+		(property "Datasheet" ""
+			(at 240.03 81.28 0)
+			(hide yes)
+			(show_name no)
+			(do_not_autoplace no)
+			(effects
+				(font
+					(size 1.27 1.27)
+				)
+			)
+		)
+		(property "Description" "Push button switch, generic, two pins"
+			(at 240.03 86.36 0)
+			(hide yes)
+			(show_name no)
+			(do_not_autoplace no)
+			(effects
+				(font
+					(size 1.27 1.27)
+				)
+			)
+		)
+		(pin "1"
+		)
+		(pin "2"
+		)
+		(instances
+			(project "ATTN_unit"
+				(path "/a8324393-8ff7-4c89-9925-098d0efac1b8"
+					(reference "SW1")
+					(unit 1)
+				)

Commit message: Add files via upload
Parts:
- removed KY038: (no value), Custom Boards:KY038, symbol Custom Boards:KY038
- removed U1: DM-OLED096-636, Custom Boards:OLED Display - 12c - 0.96 inch, symbol DM-OLED096-636:DM-OLED096-636
- added J1: Conn_02x20_Odd_Even, Connector_PinHeader_2.54mm:PinHeader_2x20_P2.54mm_Vertical, symbol Connector_Generic:Conn_02x20_Odd_Even
- added J2: Screen Connector, Connector_PinHeader_2.54mm:PinHeader_1x08_P2.54mm_Vertical, symbol Connector:Conn_01x08_Pin
- added MK1: SPH0645LM4H, Sensor_Audio:Knowles_SPH0645LM4H-6_3.5x2.65mm, symbol Sensor_Audio:SPH0645LM4H
Connections:
- net at U4.J2_1 (3V3): now also J2.1 (VCC), MK1.5 (VDD)
- net at U4.J2_10 (IO26): now also MK1.4 (BCLK)
- net at U4.J2_9 (IO25): now also MK1.6 (DATA)
- net at SW1.2, U2.4 (GND), U4.J3_1 (GND_J3_1): now also J2.2 (GND), MK1.2 (SEL), MK1.3 (GND)
- net at U4.J3_10 (IO5): now also J2.5 (CS)
- net at U4.J3_13 (IO4): now also J2.8 (BUSY); no longer U2.3 (OUT)
- net at U4.J3_14 (IO0): now also J2.7 (RST); no longer SW1.1
- net at U4.J3_15 (IO2): now also J2.6 (DC)
- net at U4.J3_16 (IO15): now also U2.3 (OUT)
- net at U4.J3_2 (IO23): now also J2.3 (DIN)
- net at U4.J3_3 (IO22): now also MK1.1 (WS)
- net at U4.J3_6 (IO21): now also SW1.1
- net at U4.J3_9 (IO18): now also J2.4 (CLK)
